File: hardware/pager/v1/kicad/mcu.kicad_sch (KiCad schematic)
At the start: 29 parts, among them Q401 AO3400A, Q402 AO3400A, SW401 TS-1187A RESET, SW402 TS-1187A BOOT, SW403 TS-1187A UP, SW404 TS-1187A DOWN, U401 ESP32-S3-WROOM-1-N8R2

Commit message: fix(pager): resolve pre-fab review findings, rev B (#192)
TP4056 EP thermal vias; RF launch ground restored (GNSS reroutes to north corridor, DIO1 shift, 7 stitching vias); BTN_DOWN moved to RTC-capable GPIO21 via switch-role swap; board name/rev silkscreen; WROOM antenna copper keepout; battery path partially widened; accepted dispositions documented; production files regenerated with Revision B metadata.

Closes #186
Closes #187
Closes #188
Closes #189
Closes #190
Closes #191
Parts:
- SW403: value TS-1187A UP -> TS-1187A DOWN
- SW404: value TS-1187A DOWN -> TS-1187A UP
Connections:
- net BTN_DOWN: now also SW403.1 (A), SW403.2 (B), U401.23 (IO21); no longer SW404.1 (A), SW404.2 (B), U401.24 (IO47)
- net BTN_UP: now also SW404.1 (A), SW404.2 (B), U401.24 (IO47); no longer SW403.1 (A), SW403.2 (B), U401.23 (IO21)
