File: hardware/pager/v1/kicad/pager.kicad_pcb (KiCad board)
At the start: 2 copper layers, 96 x 50 mm, 97 parts, among them Q101 AO3401A, Q201 AO3401A, Q301 AO3400A, Q401 AO3400A, Q402 AO3400A, SW401 TS-1187A RESET, SW402 TS-1187A BOOT, SW403 TS-1187A UP, SW404 TS-1187A DOWN, U101 USBLC6-2SC6, U102 TP4056-42, U103 DW01A, U104 FS8205A, U105 XC6220B331MR-G, U201 LoRa1262-915TCXO, U202 ATGM336H-5N31, U401 ESP32-S3-WROOM-1-N8R2

Commit message: fix(pager): resolve pre-fab-resolvable PCB errata (via-in-pad, polarity silk, hole margin) (#185)
Other:
- board text added: "+"
- board text added: "-"

Commit message: fix(pager): resolve pre-fab review findings, rev B (#192)
TP4056 EP thermal vias; RF launch ground restored (GNSS reroutes to north corridor, DIO1 shift, 7 stitching vias); BTN_DOWN moved to RTC-capable GPIO21 via switch-role swap; board name/rev silkscreen; WROOM antenna copper keepout; battery path partially widened; accepted dispositions documented; production files regenerated with Revision B metadata.

Closes #186
Closes #187
Closes #188
Closes #189
Closes #190
Closes #191
Parts:
- SW403: value TS-1187A UP -> TS-1187A DOWN
- SW404: value TS-1187A DOWN -> TS-1187A UP
Connections:
- SW403 pad 1: /mcu/BTN_UP -> /mcu/BTN_DOWN
- SW403 pad 2: /mcu/BTN_UP -> /mcu/BTN_DOWN
- SW404 pad 1: /mcu/BTN_DOWN -> /mcu/BTN_UP
- SW404 pad 2: /mcu/BTN_DOWN -> /mcu/BTN_UP
- U401 pad 23: /mcu/BTN_UP -> /mcu/BTN_DOWN
- U401 pad 24: /mcu/BTN_DOWN -> /mcu/BTN_UP
Routing:
- net GNSS_EN: track 79.0 -> 108.8 mm
- net GNSS_RX: track 85.4 -> 108.2 mm
- net GNSS_TX: track 92.4 -> 114.1 mm
- net /mcu/BTN_UP: track 35.8 -> 50.3 mm
- net /mcu/BTN_DOWN: track 50.3 -> 35.8 mm
- net RADIO_DIO1: track 25.0 -> 25.8 mm
- net GND: vias 10 -> 23
Other:
- board text added: "BRAMBLE PAGER v1 rev B"
- board text added: "v1B"
